File: micro_puerta/A_IN_4-20mA.kicad_sch (KiCad schematic)
At the start: 9 parts, among them U3 AP63200WU

Commit message: Actualizacion
Parts:
- removed C3: 10nF, symbol Device:C
- removed C4: 100nF, symbol Device:C
- removed C5: 100pF, symbol Device:C
- removed C6, C7: 22uF, symbol Device:C
- removed L1: 6.8uH, symbol Device:L
- removed R5: 196k, symbol Device:R
- removed R6: 62k, symbol Device:R
- removed U3: AP63200WU, Package_TO_SOT_SMD:TSOT-23-6, symbol Regulator_Switching:AP63200WU
- added C10: 0.1uF, symbol Device:C
- added C11: 1uF, symbol Device:C
- added D4: 12V, symbol Device:D_Zener
- added R27: 0, symbol Device:R
- added R28, R29: 4.7K, symbol Device:R
- added U12: ~, symbol Proyecto_componente:GP8201S
Connections:
- net GND: now also C10.2, C11.2, D4.2 (A), U12.5 (GND)
- net VCC: now also U12.4 (VCC)
- new net: R27.1, U12.7 (SEL)
- new net: C11.1, R27.2, U12.8 (V5V)
- new net +3.3V: R28.1, R29.1
- new net SCLK: R28.2, U12.1 (SCLK)
- new net SDA: R29.2, U12.2 (SDA)
- new net V_An_OUT: C10.1, D4.1 (K), U12.6 (VOUT)
- no-connect marks 0 -> 1
