File: micro_puerta/untitled.kicad_sch (KiCad schematic)
At the start: 3 parts, among them U1 ESP32-S3-WROOM-1

Commit message: Actualizacion PCB
Changed lines of the file:
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@@
 	)
 	(hierarchical_label "RLY1_C"
-		(shape input)
+		(shape output)
 		(at 26.67 59.69 0)
 		(effects
@@
 	)
 	(hierarchical_label "RLY2_C"
-		(shape input)
+		(shape output)
 		(at 66.04 78.74 0)
 		(effects

Commit message: Actualizacion
Connections:
- net RS485_driver/RS485_IN: now also U1.36 (RXD0); no longer U1.37 (TXD0)
- net RS485_driver/RS485_OUT: now also U1.37 (TXD0); no longer U1.36 (RXD0)
- net OUT_4-20mA/IN_4-20mA: now reaches U1.10 (IO17)
- net Rele_IN/RELAY1_IN: now reaches U1.4 (IO4)
- net Rele_IN/RELAY2_IN: now reaches U1.5 (IO5)
Other:
- added sheet A_IN_10V (A_IN_10V.kicad_sch)
- added sheet A_IN_32V (A_IN_32V.kicad_sch)
- added sheet Ma_OUT (Ma_OUT.kicad_sch)
- added sheet NPN_IN (PNP_IN.kicad_sch)
- added sheet NPN_OUT (NPN_OUT.kicad_sch)
- added sheet OUT_4-20mA (OUT_4-20mA.kicad_sch)
- added sheet PNP_IN (PNP_IN.kicad_sch)
- added sheet PNP_OUT (PNP_OUT.kicad_sch)
- added sheet Rele_IN (Rele_IN.kicad_sch)
- added sheet V_AN_Out (V_AN_Out.kicad_sch)

Commit message: actualizacion placa
Parts:
- removed U1: ESP32-S3-WROOM-1, RF_Module:ESP32-S3-WROOM-1, symbol RF_Module:ESP32-S3-WROOM-1
- added U1: ESP32-S3-WROOM-1, PCM_Espressif:ESP32-S3-WROOM-1, symbol PCM_Espressif:ESP32-S3-WROOM-1
Connections:
- net +3.3V: now also U1.2 (3V3)
- net GND: now also U1.1 (GND), U1.40 (GND), U1.41 (GND)
- net NPN_IN/PNP_IN_OUT_1: now also U1.7 (GPIO7/TOUCH7/ADC1_CH6)
- net NPN_IN/PNP_IN_OUT_2: now also U1.6 (GPIO6/TOUCH6/ADC1_CH5)
- net NPN_OUT/NPN_OUT_IN_1: now also U1.4 (GPIO4/TOUCH4/ADC1_CH3)
- net NPN_OUT/NPN_OUT_IN_2: now also U1.5 (GPIO5/TOUCH5/ADC1_CH4)
- net OUT_4-20mA/IN_4-20mA: now also U1.39 (GPIO1/TOUCH1/ADC1_CH0)
- net PNP_OUT/PNP_OUT_IN_1: now also U1.12 (GPIO8/TOUCH8/ADC1_CH7/SUBSPICS1)
- net PNP_OUT/PNP_OUT_IN_2: now also U1.17 (GPIO9/TOUCH9/ADC1_CH8/FSPIHD/SUBSPIHD)
- net RS485_driver/RS485_IN: now also U1.36 (U0RXD/GPIO44/CLK_OUT2)
- net RS485_driver/RS485_OUT: now also U1.37 (U0TXD/GPIO43/CLK_OUT1)
- net Rele_IN/RELAY1_IN: now also U1.15 (GPIO3/TOUCH3/ADC1_CH2)
- net Rele_IN/RELAY2_IN: now also U1.38 (GPIO2/TOUCH2/ADC1_CH1)
- net at C1.1, R1.2: now also U1.3 (EN)
- new net PNP_IN/PNP_IN_IN_1: U1.18 (GPIO10/TOUCH10/ADC1_CH9/FSPICS0/FSPIIO4/SUBSPICS0)
- new net PNP_IN/PNP_IN_IN_2: U1.19 (GPIO11/TOUCH11/ADC2_CH0/FSPID/FSPIIO5/SUBSPID)
Other:
- sheet Ma_OUT ports: added none; removed A0, A1, A2
- moved on the sheet: C1, R1

Commit message: nueva actualizacion
Parts:
- added R33: 2.2K, symbol Device:R
Connections:
- net +3.3V: now also R33.1
- net A_IN_10V/10V_A_IN_OUT: now also U1.20 (GPIO12/TOUCH12/ADC2_CH1/FSPICLK/FSPIIO6/SUBSPICLK)
- net A_IN_32V/32v_A_IN_OUT: now also U1.21 (GPIO13/TOUCH13/ADC2_CH2/FSPIQ/FSPIIO7/SUBSPIQ)
- net Ma_OUT/SDA: now also U1.35 (MTMS/GPIO42), R33.2
- net Ma_OUT/SLCLK: now also U1.34 (MTDI/GPIO41/CLK_OUT1)
