File: micro_puerta/untitled.kicad_sch (KiCad schematic)
At the start: 4 parts, among them U1 ESP32-S3-WROOM-1

Commit message: Actualizacion 5
Connections:
- net NPN_OUT/NPN_OUT_IN_1: now also U1.19 (GPIO11/TOUCH11/ADC2_CH0/FSPID/FSPIIO5/SUBSPID)
- net NPN_OUT/NPN_OUT_IN_2: now also U1.20 (GPIO12/TOUCH12/ADC2_CH1/FSPICLK/FSPIIO6/SUBSPICLK)
Changed lines of the file:
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@@
+	(wire
+		(pts
+			(xy 209.55 135.89) (xy 198.12 135.89)
+		)
+		(stroke
+			(width 0)
+			(type default)
+		)
+	)
 	(wire
 		(pts
@@
 	(wire
 		(pts
-			(xy 261.62 135.89) (xy 257.81 135.89)
+			(xy 255.27 135.89) (xy 246.38 135.89)
 		)
 		(stroke
@@
 	(wire
 		(pts
-			(xy 261.62 139.7) (xy 257.81 139.7)
+			(xy 255.27 139.7) (xy 246.38 139.7)
 		)
 		(stroke
@@
 	(wire
 		(pts
+			(xy 194.31 81.28) (xy 186.69 81.28)
+		)
+		(stroke
+			(width 0)
+			(type default)
+		)
+	)
+	(wire
+		(pts
+			(xy 194.31 139.7) (xy 194.31 81.28)
+		)
+		(stroke
+			(width 0)
+			(type default)
+		)
+	)
+	(wire
+		(pts
 			(xy 238.76 77.47) (xy 243.84 77.47)
 		)
@@
 	(wire
 		(pts
+			(xy 209.55 139.7) (xy 194.31 139.7)
+		)
+		(stroke
+			(width 0)
+			(type default)
+		)
+	)
+	(wire
+		(pts
 			(xy 238.76 72.39) (xy 243.84 72.39)
 		)
@@
 	(wire
 		(pts
+			(xy 198.12 78.74) (xy 186.69 78.74)
+		)
+		(stroke
+			(width 0)
+			(type default)
+		)
+	)
+	(wire
+		(pts
 			(xy 95.25 85.09) (xy 95.25 58.42)
 		)
@@
 		(pts
 			(xy 213.36 43.18) (xy 215.9 43.18)
+		)
+		(stroke
+			(width 0)
+			(type default)
+		)
+	)
+	(wire
+		(pts
+			(xy 198.12 135.89) (xy 198.12 78.74)
 		)
 		(stroke
@@
 	(hierarchical_label "NPN_OUT_1"
 		(shape output)
-		(at 261.62 135.89 0)
+		(at 255.27 135.89 0)
 		(effects
 			(font
@@
 	(hierarchical_label "NPN_OUT_2"
 		(shape output)
-		(at 261.62 139.7 0)
+		(at 255.27 139.7 0)
 		(effects
 			(font
@@
 	)
 	(sheet
-		(at 220.98 133.35)
-		(size 36.83 12.7)
+		(at 209.55 133.35)
+		(size 36.83 8.89)
 		(exclude_from_sim no)
 		(in_bom yes)
@@
 		)
 		(property "Sheetname" "NPN_OUT"
-			(at 220.98 132.6384 0)
+			(at 209.55 132.6384 0)
 			(effects
 				(font
@@
 		)
 		(property "Sheetfile" "NPN_OUT.kicad_sch"
-			(at 220.98 146.6346 0)
+			(at 209.55 142.8246 0)
 			(effects
 				(font
@@
 		)
 		(pin "NPN_OUT_IN_1" output
-			(at 220.98 135.89 180)
+			(at 209.55 135.89 180)
 			(effects
 				(font
@@
 		)
 		(pin "NPN_OUT_IN_2" output
-			(at 220.98 139.7 180)
+			(at 209.55 139.7 180)
 			(effects
 				(font
@@
 		)
 		(pin "NPN_OUT_OUT_1" output
-			(at 257.81 135.89 0)
+			(at 246.38 135.89 0)
 			(effects
 				(font
@@
 		)
 		(pin "NPN_OUT_OUT_2" output
-			(at 257.81 139.7 0)
-			(effects
-				(font
+			(at 246.38 139.7 0)
+			(effects
+				(font

Commit message: Actualizacion 6
Connections:
- net OUT_4-20mA/IN_4-20mA is gone; now on net NPN_OUT/NPN_OUT_IN_1: U1.14 (GPIO20/U1CTS/ADC2_CH9/CLK_OUT1/USB_D+)
- net NPN_OUT/NPN_OUT_IN_1: now also U1.36 (U0RXD/GPIO44/CLK_OUT2); no longer U1.19 (GPIO11/TOUCH11/ADC2_CH0/FSPID/FSPIIO5/SUBSPID)
- net NPN_OUT/NPN_OUT_IN_2: now also U1.37 (U0TXD/GPIO43/CLK_OUT1); no longer U1.20 (GPIO12/TOUCH12/ADC2_CH1/FSPICLK/FSPIIO6/SUBSPICLK)
- net PNP_OUT/PNP_OUT_IN_1: now also U1.38 (GPIO2/TOUCH2/ADC1_CH1)
- net PNP_OUT/PNP_OUT_IN_2: now also U1.39 (GPIO1/TOUCH1/ADC1_CH0)
Other:
- removed sheet Power_supply
