File: micro_puerta/A_IN_10V.kicad_sch (KiCad schematic)
At the start: 3 parts

Commit message: Actualizacion 4 de proyecto
Parts:
- C9: renamed from C8; footprint (none) -> Capacitor_SMD:C_0201_0603Metric
- R22: renamed from R11; footprint (none) -> Resistor_SMD:R_0201_0603Metric
- R23: renamed from R12; footprint (none) -> Resistor_SMD:R_0201_0603Metric
Changed lines of the file:
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@@
 		(dnp no)
 		(fields_autoplaced yes)
-		(property "Reference" "R11"
+		(property "Reference" "R22"
 			(at 132.08 86.3599 0)
 			(effects
@@
 			)
 		)
-		(property "Footprint" ""
+		(property "Footprint" "Resistor_SMD:R_0201_0603Metric"
 			(at 127.762 87.63 90)
 			(effects
@@
 			(project "micro_puerta"
 				(path "/ab2f26d1-d065-4d9e-8f9a-0ccfc45c4b5b/f046d5e0-b81e-417d-b1cc-4f018da2dc07/fae1c8b8-9712-4877-851a-b7d5d9648c1b"
-					(reference "R11")
+					(reference "R22")
 					(unit 1)
 				)
@@
 		(dnp no)
 		(fields_autoplaced yes)
-		(property "Reference" "C8"
+		(property "Reference" "C9"
 			(at 143.51 99.0599 0)
 			(effects
@@
 			)
 		)
-		(property "Footprint" ""
+		(property "Footprint" "Capacitor_SMD:C_0201_0603Metric"
 			(at 140.6652 104.14 0)
 			(effects
@@
 			(project "micro_puerta"
 				(path "/ab2f26d1-d065-4d9e-8f9a-0ccfc45c4b5b/f046d5e0-b81e-417d-b1cc-4f018da2dc07/fae1c8b8-9712-4877-851a-b7d5d9648c1b"
-					(reference "C8")
+					(reference "C9")
 					(unit 1)
 				)
@@
 		(dnp no)
 		(fields_autoplaced yes)
-		(property "Reference" "R12"
+		(property "Reference" "R23"
 			(at 132.08 99.0599 0)
 			(effects
@@
 			)
 		)
-		(property "Footprint" ""
+		(property "Footprint" "Resistor_SMD:R_0201_0603Metric"
 			(at 127.762 100.33 90)
 			(effects
@@
 			(project "micro_puerta"
 				(path "/ab2f26d1-d065-4d9e-8f9a-0ccfc45c4b5b/f046d5e0-b81e-417d-b1cc-4f018da2dc07/fae1c8b8-9712-4877-851a-b7d5d9648c1b"
-					(reference "R12")
+					(reference "R23")
 					(unit 1)
 				)
@@
 		(dnp no)
 		(fields_autoplaced yes)
-		(property "Reference" "#PWR025"
+		(property "Reference" "#PWR042"
 			(at 129.54 115.57 0)
 			(effects
@@
 			(project "micro_puerta"
 				(path "/ab2f26d1-d065-4d9e-8f9a-0ccfc45c4b5b/f046d5e0-b81e-417d-b1cc-4f018da2dc07/fae1c8b8-9712-4877-851a-b7d5d9648c1b"
-					(reference "#PWR025")
-					(unit 1)
-				)
+					(reference "#PWR042")
+					(unit 1)
+				)
