File: micro_puerta/NPN_OUT.kicad_sch (KiCad schematic)
At the start: 8 parts, among them Q1 NCV8402xST, Q2 NCV8402xST, U10 LTV-357T, U11 LTV-357T

Commit message: Actualizacion 4 de proyecto
Parts:
- removed R23, R25: 100, symbol Device:R
- removed R24, R26: R, symbol Device:R
- removed U10, U11: LTV-357T, Package_SO:SO-4_4.4x3.6mm_P2.54mm, symbol Isolator:LTV-357T
Connections:
- net NPN_OUT_IN_1: now also Q1.1 (G)
- net NPN_OUT_IN_2: now also Q2.1 (G)
- net GNDPWR renamed GND
