File: micro_puerta/PNP_IN.kicad_sch (KiCad schematic)
At the start: 6 parts, among them U5 LTV-357T, U6 LTV-357T

Commit message: actualizacion placa
Parts:
- renumbered R19 to R13, R20 to R14, R9 to R7, R10 to R8, U5 to U4, U6 to U7
Changed lines of the file:
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@@
 		(dnp no)
 		(fields_autoplaced yes)
-		(property "Reference" "U6"
+		(property "Reference" "U7"
 			(at 182.88 85.09 0)
 			(effects
@@
 					(unit 1)
 				)
+				(path "/ab2f26d1-d065-4d9e-8f9a-0ccfc45c4b5b/f046d5e0-b81e-417d-b1cc-4f018da2dc07/c9a7c916-5eae-47c8-9edb-203b51fa0814"
+					(reference "U7")
+					(unit 1)
+				)
 			)
 		)
@@
 		(dnp no)
 		(fields_autoplaced yes)
-		(property "Reference" "R20"
+		(property "Reference" "R14"
 			(at 199.39 82.5499 0)
 			(effects
@@
 					(unit 1)
 				)
+				(path "/ab2f26d1-d065-4d9e-8f9a-0ccfc45c4b5b/f046d5e0-b81e-417d-b1cc-4f018da2dc07/c9a7c916-5eae-47c8-9edb-203b51fa0814"
+					(reference "R14")
+					(unit 1)
+				)
 			)
 		)
@@
 		(dnp no)
 		(fields_autoplaced yes)
-		(property "Reference" "#PWR038"
+		(property "Reference" "#PWR0103"
 			(at 196.85 81.28 0)
 			(effects
@@
 					(unit 1)
 				)
+				(path "/ab2f26d1-d065-4d9e-8f9a-0ccfc45c4b5b/f046d5e0-b81e-417d-b1cc-4f018da2dc07/c9a7c916-5eae-47c8-9edb-203b51fa0814"
+					(reference "#PWR0103")
+					(unit 1)
+				)
 			)
 		)
@@
 		(dnp no)
 		(fields_autoplaced yes)
-		(property "Reference" "#PWR024"
+		(property "Reference" "#PWR0104"
 			(at 85.09 102.87 0)
 			(effects
@@
 					(unit 1)
 				)
+				(path "/ab2f26d1-d065-4d9e-8f9a-0ccfc45c4b5b/f046d5e0-b81e-417d-b1cc-4f018da2dc07/c9a7c916-5eae-47c8-9edb-203b51fa0814"
+					(reference "#PWR0104")
+					(unit 1)
+				)
 			)
 		)
@@
 		(dnp no)
 		(fields_autoplaced yes)
-		(property "Reference" "R9"
+		(property "Reference" "R7"
 			(at 78.74 85.09 90)
 			(effects
@@
 					(unit 1)
 				)
+				(path "/ab2f26d1-d065-4d9e-8f9a-0ccfc45c4b5b/f046d5e0-b81e-417d-b1cc-4f018da2dc07/c9a7c916-5eae-47c8-9edb-203b51fa0814"
+					(reference "R7")
+					(unit 1)
+				)
 			)
 		)
@@
 		(dnp no)
 		(fields_autoplaced yes)
-		(property "Reference" "R19"
+		(property "Reference" "R13"
 			(at 163.83 85.09 90)
 			(effects
@@
 					(unit 1)
 				)
+				(path "/ab2f26d1-d065-4d9e-8f9a-0ccfc45c4b5b/f046d5e0-b81e-417d-b1cc-4f018da2dc07/c9a7c916-5eae-47c8-9edb-203b51fa0814"
+					(reference "R13")
+					(unit 1)
+				)
 			)
 		)
@@
 		(dnp no)
 		(fields_autoplaced yes)
-		(property "Reference" "#PWR036"
+		(property "Reference" "#PWR0102"
 			(at 170.18 102.87 0)
 			(effects
@@
 					(unit 1)
 				)
+				(path "/ab2f26d1-d065-4d9e-8f9a-0ccfc45c4b5b/f046d5e0-b81e-417d-b1cc-4f018da2dc07/c9a7c916-5eae-47c8-9edb-203b51fa0814"
+					(reference "#PWR0102")
+					(unit 1)
+				)
 			)
 		)
@@
 		(dnp no)
 		(fields_autoplaced yes)
-		(property "Reference" "#PWR035"
+		(property "Reference" "#PWR0106"
 			(at 111.76 81.28 0)
 			(effects
@@
 					(unit 1)
 				)
+				(path "/ab2f26d1-d065-4d9e-8f9a-0ccfc45c4b5b/f046d5e0-b81e-417d-b1cc-4f018da2dc07/c9a7c916-5eae-47c8-9edb-203b51fa0814"
+					(reference "#PWR0106")
+					(unit 1)
+				)
 			)
 		)
@@
 		(dnp no)
 		(fields_autoplaced yes)
-		(property "Reference" "#PWR027"
+		(property "Reference" "#PWR0101"
 			(at 110.49 105.41 0)
 			(effects
@@
 					(unit 1)
 				)
+				(path "/ab2f26d1-d065-4d9e-8f9a-0ccfc45c4b5b/f046d5e0-b81e-417d-b1cc-4f018da2dc07/c9a7c916-5eae-47c8-9edb-203b51fa0814"
+					(reference "#PWR0101")
+					(unit 1)
+				)
 			)
 		)
@@
 		(dnp no)
 		(fields_autoplaced yes)
-		(property "Reference" "U5"
+		(property "Reference" "U4"
 			(at 97.79 85.09 0)
 			(effects
@@
 					(unit 1)
 				)
+				(path "/ab2f26d1-d065-4d9e-8f9a-0ccfc45c4b5b/f046d5e0-b81e-417d-b1cc-4f018da2dc07/c9a7c916-5eae-47c8-9edb-203b51fa0814"
+					(reference "U4")
+					(unit 1)
+				)
 			)
 		)
@@
 		(dnp no)
 		(fields_autoplaced yes)
-		(property "Reference" "R10"
+		(property "Reference" "R8"
 			(at 114.3 82.5499 0)
 			(effects
@@
 					(unit 1)
 				)
+				(path "/ab2f26d1-d065-4d9e-8f9a-0ccfc45c4b5b/f046d5e0-b81e-417d-b1cc-4f018da2dc07/c9a7c916-5eae-47c8-9edb-203b51fa0814"
+					(reference "R8")
+					(unit 1)
+				)
 			)
 		)
@@
 		(dnp no)
 		(fields_autoplaced yes)
-		(property "Reference" "#PWR037"
+		(property "Reference" "#PWR0105"
 			(at 195.58 105.41 0)
 			(effects
@@
 					(unit 1)
 				)
+				(path "/ab2f26d1-d065-4d9e-8f9a-0ccfc45c4b5b/f046d5e0-b81e-417d-b1cc-4f018da2dc07/c9a7c916-5eae-47c8-9edb-203b51fa0814"
+					(reference "#PWR0105")
+					(unit 1)
+				)

Commit message: Actualizacion 4 de proyecto
Parts:
- removed R13, R7: 910, symbol Device:R
- removed R14, R8: 412, symbol Device:R
- removed U4, U7: LTV-357T, Package_SO:SO-4_4.4x3.6mm_P2.54mm, symbol Isolator:LTV-357T
- added R16, R18: 910, Resistor_SMD:R_0201_0603Metric, symbol Device:R
- added R17, R19: 412, Resistor_SMD:R_0201_0603Metric, symbol Device:R
- added U10, U9: LTV-357T, Package_SO:SO-4_4.4x3.6mm_P2.54mm, symbol Isolator:LTV-357T
Connections:
- net +3.3V: now also U10.4, U9.4
- net GND: now also R17.2, R19.2
- net GNDPWR: now also U10.2, U9.2
- net PNP_IN_IN_1: now also R16.1
- net PNP_IN_IN_2: now also R18.1
- net PNP_IN_OUT_1: now also R17.1, U9.3
- net PNP_IN_OUT_2: now also R19.1, U10.3
- new net: R18.2, U10.1
- new net: R16.2, U9.1
