File: micro_puerta/RS485_driver.kicad_sch (KiCad schematic)
At the start: 0 parts

Commit message: Actualizacion
Parts:
- added D1: SM712_SOT23, Package_TO_SOT_SMD:SOT-23, symbol Diode:SM712_SOT23
- added R2, R3: 120, symbol Device:R
- added U2: ~, Proyecto_componente:RSM3485ECHT, symbol Proyecto_componente:RSM3485ECHT
Connections:
- net RS485_A: now also D1.2 (A2), R2.2
- net RS485_B: now also D1.1 (A1), R3.2
- net RS485_IN: now also U2.4 (RXD)
- net RS485_OUT: now also U2.3 (TXD)
- new net: R2.1, U2.6 (B)
- new net: R3.1, U2.7 (A)
- new net +3.3V: U2.1 (VCC)
- new net GND: D1.3 (common), U2.2 (GND)

Commit message: Actualizacion 4 de proyecto
Parts:
- R5: renamed from R2; footprint (none) -> Resistor_SMD:R_0201_0603Metric
- R6: renamed from R3; footprint (none) -> Resistor_SMD:R_0201_0603Metric
- renumbered U2 to U3
Changed lines of the file:
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@@
 		(on_board yes)
 		(dnp no)
-		(property "Reference" "R2"
+		(property "Reference" "R5"
 			(at 171.45 79.248 90)
 			(effects
@@
 			)
 		)
-		(property "Footprint" ""
+		(property "Footprint" "Resistor_SMD:R_0201_0603Metric"
 			(at 171.45 83.058 90)
 			(effects
@@
 			(project ""
 				(path "/ab2f26d1-d065-4d9e-8f9a-0ccfc45c4b5b/f046d5e0-b81e-417d-b1cc-4f018da2dc07/0c97fc1b-5dea-4bbd-a681-4ace400501e9"
-					(reference "R2")
+					(reference "R5")
 					(unit 1)
 				)
@@
 		(on_board yes)
 		(dnp no)
-		(property "Reference" "R3"
+		(property "Reference" "R6"
 			(at 171.45 86.614 90)
 			(effects
@@
 			)
 		)
-		(property "Footprint" ""
+		(property "Footprint" "Resistor_SMD:R_0201_0603Metric"
 			(at 171.45 90.678 90)
 			(effects
@@
 			(project ""
 				(path "/ab2f26d1-d065-4d9e-8f9a-0ccfc45c4b5b/f046d5e0-b81e-417d-b1cc-4f018da2dc07/0c97fc1b-5dea-4bbd-a681-4ace400501e9"
-					(reference "R3")
+					(reference "R6")
 					(unit 1)
 				)
@@
 		(dnp no)
 		(fields_autoplaced yes)
-		(property "Reference" "U2"
+		(property "Reference" "U3"
 			(at 145.415 69.85 0)
 			(effects
@@
 			(project ""
 				(path "/ab2f26d1-d065-4d9e-8f9a-0ccfc45c4b5b/f046d5e0-b81e-417d-b1cc-4f018da2dc07/0c97fc1b-5dea-4bbd-a681-4ace400501e9"
-					(reference "U2")
+					(reference "U3")
 					(unit 1)
 				)
@@
 		(dnp no)
 		(fields_autoplaced yes)
-		(property "Reference" "#PWR014"
+		(property "Reference" "#PWR018"
 			(at 121.92 81.28 0)
 			(effects
@@
 			(project ""
 				(path "/ab2f26d1-d065-4d9e-8f9a-0ccfc45c4b5b/f046d5e0-b81e-417d-b1cc-4f018da2dc07/0c97fc1b-5dea-4bbd-a681-4ace400501e9"
-					(reference "#PWR014")
+					(reference "#PWR018")
 					(unit 1)
 				)
@@
 		(dnp no)
 		(fields_autoplaced yes)
-		(property "Reference" "#PWR015"
+		(property "Reference" "#PWR019"
 			(at 186.69 113.03 0)
 			(effects
@@
 			(project ""
 				(path "/ab2f26d1-d065-4d9e-8f9a-0ccfc45c4b5b/f046d5e0-b81e-417d-b1cc-4f018da2dc07/0c97fc1b-5dea-4bbd-a681-4ace400501e9"
-					(reference "#PWR015")
+					(reference "#PWR019")
 					(unit 1)
 				)
@@
 		(dnp no)
 		(fields_autoplaced yes)
-		(property "Reference" "#PWR013"
+		(property "Reference" "#PWR017"
 			(at 123.19 76.2 0)
 			(effects
@@
 			(project ""
 				(path "/ab2f26d1-d065-4d9e-8f9a-0ccfc45c4b5b/f046d5e0-b81e-417d-b1cc-4f018da2dc07/0c97fc1b-5dea-4bbd-a681-4ace400501e9"
-					(reference "#PWR013")
-					(unit 1)
-				)
+					(reference "#PWR017")
+					(unit 1)
+				)
