File: micro_puerta/Rele_IN.kicad_sch (KiCad schematic)
At the start: 3 parts, among them K1 SANYOU_SRD_Form_C, K2 SANYOU_SRD_Form_C

Commit message: Actualizacion 4 de proyecto
Parts:
- U4: renamed from U14; footprint (none) -> Proyecto_componente:LK1802
Changed lines of the file:
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@@
 		(dnp no)
 		(fields_autoplaced yes)
-		(property "Reference" "U14"
+		(property "Reference" "U4"
 			(at 97.79 96.52 0)
 			(effects
@@
 			)
 		)
-		(property "Footprint" ""
+		(property "Footprint" "Proyecto_componente:LK1802"
 			(at 97.79 106.68 0)
 			(effects
@@
 			(project ""
 				(path "/ab2f26d1-d065-4d9e-8f9a-0ccfc45c4b5b/f046d5e0-b81e-417d-b1cc-4f018da2dc07/5b0695e4-d78f-4e3e-8724-d3eb950f912a"
-					(reference "U14")
+					(reference "U4")
 					(unit 1)
 				)
@@
 		(dnp no)
 		(fields_autoplaced yes)
-		(property "Reference" "#PWR055"
+		(property "Reference" "#PWR021"
 			(at 85.09 113.03 0)
 			(effects
@@
 			(project ""
 				(path "/ab2f26d1-d065-4d9e-8f9a-0ccfc45c4b5b/f046d5e0-b81e-417d-b1cc-4f018da2dc07/5b0695e4-d78f-4e3e-8724-d3eb950f912a"
-					(reference "#PWR055")
+					(reference "#PWR021")
 					(unit 1)
 				)
@@
 		(dnp no)
 		(fields_autoplaced yes)
-		(property "Reference" "#PWR017"
+		(property "Reference" "#PWR023"
 			(at 123.19 52.07 0)
 			(effects
@@
 			(project ""
 				(path "/ab2f26d1-d065-4d9e-8f9a-0ccfc45c4b5b/f046d5e0-b81e-417d-b1cc-4f018da2dc07/5b0695e4-d78f-4e3e-8724-d3eb950f912a"
-					(reference "#PWR017")
+					(reference "#PWR023")
 					(unit 1)
 				)
@@
 		(dnp no)
 		(fields_autoplaced yes)
-		(property "Reference" "#PWR054"
+		(property "Reference" "#PWR022"
 			(at 110.49 107.95 0)
 			(effects
@@
 			(project ""
 				(path "/ab2f26d1-d065-4d9e-8f9a-0ccfc45c4b5b/f046d5e0-b81e-417d-b1cc-4f018da2dc07/5b0695e4-d78f-4e3e-8724-d3eb950f912a"
-					(reference "#PWR054")
+					(reference "#PWR022")
 					(unit 1)
 				)
@@
 		(dnp no)
 		(fields_autoplaced yes)
-		(property "Reference" "#PWR018"
+		(property "Reference" "#PWR024"
 			(at 181.61 52.07 0)
 			(effects
@@
 			(project "micro_puerta"
 				(path "/ab2f26d1-d065-4d9e-8f9a-0ccfc45c4b5b/f046d5e0-b81e-417d-b1cc-4f018da2dc07/5b0695e4-d78f-4e3e-8724-d3eb950f912a"
-					(reference "#PWR018")
-					(unit 1)
-				)
+					(reference "#PWR024")
+					(unit 1)
+				)
