File: micro_puerta/power_supply.kicad_sch (KiCad schematic)
At the start: 9 parts, among them U3 AP63200WU

Commit message: Actualizacion 4 de proyecto
Parts:
- renumbered C3 to C2, C4 to C3, C5 to C4, C6 to C5, C7 to C6, R5 to R3, R6 to R4, U3 to U2
Changed lines of the file:
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@@
 		(dnp no)
 		(fields_autoplaced yes)
-		(property "Reference" "C4"
+		(property "Reference" "C3"
 			(at 77.47 60.96 90)
 			(effects
@@
 			(project "micro_puerta"
 				(path "/ab2f26d1-d065-4d9e-8f9a-0ccfc45c4b5b/f046d5e0-b81e-417d-b1cc-4f018da2dc07/a4982cd6-d21b-4306-bf3a-2b740cc8f4b8"
-					(reference "C4")
+					(reference "C3")
 					(unit 1)
 				)
@@
 		(dnp no)
 		(fields_autoplaced yes)
-		(property "Reference" "#PWR022"
+		(property "Reference" "#PWR016"
 			(at 125.73 128.27 0)
 			(effects
@@
 			(project "micro_puerta"
 				(path "/ab2f26d1-d065-4d9e-8f9a-0ccfc45c4b5b/f046d5e0-b81e-417d-b1cc-4f018da2dc07/a4982cd6-d21b-4306-bf3a-2b740cc8f4b8"
-					(reference "#PWR022")
+					(reference "#PWR016")
 					(unit 1)
 				)
@@
 		(dnp no)
 		(fields_autoplaced yes)
-		(property "Reference" "R6"
+		(property "Reference" "R4"
 			(at 106.68 95.2499 0)
 			(effects
@@
 			(project ""
 				(path "/ab2f26d1-d065-4d9e-8f9a-0ccfc45c4b5b/f046d5e0-b81e-417d-b1cc-4f018da2dc07/a4982cd6-d21b-4306-bf3a-2b740cc8f4b8"
-					(reference "R6")
+					(reference "R4")
 					(unit 1)
 				)
@@
 		(dnp no)
 		(fields_autoplaced yes)
-		(property "Reference" "C6"
+		(property "Reference" "C5"
 			(at 121.92 72.3899 0)
 			(effects
@@
 			(project "micro_puerta"
 				(path "/ab2f26d1-d065-4d9e-8f9a-0ccfc45c4b5b/f046d5e0-b81e-417d-b1cc-4f018da2dc07/a4982cd6-d21b-4306-bf3a-2b740cc8f4b8"
-					(reference "C6")
+					(reference "C5")
 					(unit 1)
 				)
@@
 		(dnp no)
 		(fields_autoplaced yes)
-		(property "Reference" "#PWR020"
+		(property "Reference" "#PWR014"
 			(at 35.56 85.09 0)
 			(effects
@@
 			(project ""
 				(path "/ab2f26d1-d065-4d9e-8f9a-0ccfc45c4b5b/f046d5e0-b81e-417d-b1cc-4f018da2dc07/a4982cd6-d21b-4306-bf3a-2b740cc8f4b8"
-					(reference "#PWR020")
+					(reference "#PWR014")
 					(unit 1)
 				)
@@
 		(dnp no)
 		(fields_autoplaced yes)
-		(property "Reference" "R5"
+		(property "Reference" "R3"
 			(at 106.68 82.5499 0)
 			(effects
@@
 			(project ""
 				(path "/ab2f26d1-d065-4d9e-8f9a-0ccfc45c4b5b/f046d5e0-b81e-417d-b1cc-4f018da2dc07/a4982cd6-d21b-4306-bf3a-2b740cc8f4b8"
-					(reference "R5")
+					(reference "R3")
 					(unit 1)
 				)
@@
 		(dnp no)
 		(fields_autoplaced yes)
-		(property "Reference" "#PWR019"
+		(property "Reference" "#PWR013"
 			(at 35.56 63.5 0)
 			(effects
@@
 			(project ""
 				(path "/ab2f26d1-d065-4d9e-8f9a-0ccfc45c4b5b/f046d5e0-b81e-417d-b1cc-4f018da2dc07/a4982cd6-d21b-4306-bf3a-2b740cc8f4b8"
-					(reference "#PWR019")
+					(reference "#PWR013")
 					(unit 1)
 				)
@@
 		(dnp no)
 		(fields_autoplaced yes)
-		(property "Reference" "C5"
+		(property "Reference" "C4"
 			(at 92.71 69.85 90)
 			(effects
@@
 			(project "micro_puerta"
 				(path "/ab2f26d1-d065-4d9e-8f9a-0ccfc45c4b5b/f046d5e0-b81e-417d-b1cc-4f018da2dc07/a4982cd6-d21b-4306-bf3a-2b740cc8f4b8"
-					(reference "C5")
+					(reference "C4")
 					(unit 1)
 				)
@@
 		(dnp no)
 		(fields_autoplaced yes)
-		(property "Reference" "#PWR021"
+		(property "Reference" "#PWR015"
 			(at 59.69 86.36 0)
 			(effects
@@
 			(project "micro_puerta"
 				(path "/ab2f26d1-d065-4d9e-8f9a-0ccfc45c4b5b/f046d5e0-b81e-417d-b1cc-4f018da2dc07/a4982cd6-d21b-4306-bf3a-2b740cc8f4b8"
-					(reference "#PWR021")
+					(reference "#PWR015")
 					(unit 1)
 				)
@@
 		(dnp no)
 		(fields_autoplaced yes)
-		(property "Reference" "C7"
+		(property "Reference" "C6"
 			(at 137.16 72.3899 0)
 			(effects
@@
 			(project "micro_puerta"
 				(path "/ab2f26d1-d065-4d9e-8f9a-0ccfc45c4b5b/f046d5e0-b81e-417d-b1cc-4f018da2dc07/a4982cd6-d21b-4306-bf3a-2b740cc8f4b8"
-					(reference "C7")
+					(reference "C6")
 					(unit 1)
 				)
@@
 		(dnp no)
 		(fields_autoplaced yes)
-		(property "Reference" "U3"
+		(property "Reference" "U2"
 			(at 59.69 58.42 0)
 			(effects
@@
 			(project ""
 				(path "/ab2f26d1-d065-4d9e-8f9a-0ccfc45c4b5b/f046d5e0-b81e-417d-b1cc-4f018da2dc07/a4982cd6-d21b-4306-bf3a-2b740cc8f4b8"
-					(reference "U3")
+					(reference "U2")
 					(unit 1)
 				)
@@
 		(dnp no)
 		(fields_autoplaced yes)
-		(property "Reference" "C3"
+		(property "Reference" "C2"
 			(at 39.37 69.8499 0)
 			(effects
@@
 			(project ""
 				(path "/ab2f26d1-d065-4d9e-8f9a-0ccfc45c4b5b/f046d5e0-b81e-417d-b1cc-4f018da2dc07/a4982cd6-d21b-4306-bf3a-2b740cc8f4b8"
-					(reference "C3")
-					(unit 1)
-				)
+					(reference "C2")
+					(unit 1)
+				)
