File: micro_puerta/micro_puerta.kicad_pcb (KiCad board)
At the start: 2 copper layers, 16 parts, among them J1 Entrada NPN, J10 Screw_Terminal_01x02, J11 Screw_Terminal_01x02, J2 Entradas PNP, J3 Entrada An 0-32V, J4 Entrada An 0-10V, J5 Relay, J6 Entrada An 4-20mA, J7 Salida An 4-20mA, J8 Salida An 0-10V, J9 RS485, U1 ESP32-S3-WROOM-1

Commit message: Actualizacion 4 de proyecto
Parts:
- removed the REF** at (230.0, 55.5)
- removed the REF** at (60.0, 155.5)
- added C7: 100nF, Capacitor_SMD:C_0201_0603Metric, F.Cu at (113.0, 76.0)
- added C8: 100nF, Capacitor_SMD:C_0201_0603Metric, F.Cu at (117.5, 84.0)
- added C9: 100nF, Capacitor_SMD:C_0201_0603Metric, F.Cu at (115.0, 78.5)
- added D1: SM712_SOT23, Package_TO_SOT_SMD:SOT-23, F.Cu at (125.5, 134.4)
- added D2: SMF24A, Diode_SMD:D_SMF, F.Cu at (234.6, 113.2)
- added K1: SANYOU_SRD_Form_C, Relay_THT:Relay_SPDT_SANYOU_SRD_Series_Form_C, F.Cu at (88.0, 120.5)
- added K2: SANYOU_SRD_Form_C, Relay_THT:Relay_SPDT_SANYOU_SRD_Series_Form_C, F.Cu at (105.0, 120.5)
- added Q1: NCV8402xST, Package_TO_SOT_SMD:SOT-223, F.Cu at (139.0, 132.5)
- added Q2: NCV8402xST, Package_TO_SOT_SMD:SOT-223, F.Cu at (200.2, 72.2)
- added Q3: NCV8402xST, Package_TO_SOT_SMD:SOT-223, F.Cu at (209.0, 113.5)
- added Q4: NCV8402xST, Package_TO_SOT_SMD:SOT-223, F.Cu at (214.9, 124.0)
- added R10: 910, Resistor_SMD:R_0201_0603Metric, F.Cu at (141.7, 88.0)
- added R11: 412, Resistor_SMD:R_0201_0603Metric, F.Cu at (141.7, 86.5)
- added R16: 910, Resistor_SMD:R_0201_0603Metric, F.Cu at (127.7, 88.5)
- added R17: 412, Resistor_SMD:R_0201_0603Metric, F.Cu at (127.7, 90.2)
- added R18: 910, Resistor_SMD:R_0201_0603Metric, F.Cu at (127.7, 86.8)
- added R19: 412, Resistor_SMD:R_0201_0603Metric, F.Cu at (127.5, 91.8)
- added R20: 160K, Resistor_SMD:R_0201_0603Metric, F.Cu at (117.5, 85.5)
- added R21: 13K, Resistor_SMD:R_0201_0603Metric, F.Cu at (117.7, 87.0)
- added R22: 51K, Resistor_SMD:R_0201_0603Metric, F.Cu at (115.0, 80.0)
- added R23: 16K, Resistor_SMD:R_0201_0603Metric, F.Cu at (115.0, 81.5)
- added R5: 120, Resistor_SMD:R_0201_0603Metric, F.Cu at (126.5, 138.2)
- added R6: 120, Resistor_SMD:R_0201_0603Metric, F.Cu at (124.5, 138.2)
- added R7: 120, Resistor_SMD:R_0201_0603Metric, F.Cu at (113.0, 77.5)
- added R8: 910, Resistor_SMD:R_0201_0603Metric, F.Cu at (141.7, 89.5)
- added R9: 412, Resistor_SMD:R_0201_0603Metric, F.Cu at (141.7, 85.0)
- added REF**: MountingHole_2.1mm, MountingHole:MountingHole_2.1mm, F.Cu at (169.0, 82.0)
- added REF**: MountingHole_2.1mm, MountingHole:MountingHole_2.1mm, F.Cu at (84.0, 132.0)
- added U10: LTV-357T, Package_SO:SO-4_4.4x3.6mm_P2.54mm, F.Cu at (129.0, 83.5)
- added U2: AP63200WU, Package_TO_SOT_SMD:TSOT-23-6, F.Cu at (234.2, 119.2)
- added U3: ~, Proyecto_componente:RSM3485ECHT, F.Cu at (128.5, 114.5)
- added U4: ~, Proyecto_componente:LK1802, F.Cu at (99.0, 99.0)
- added U5: LTV-357T, Package_SO:SO-4_4.4x3.6mm_P2.54mm, F.Cu at (219.8, 96.7)
- added U5: LTV-357T, Package_SO:SO-4_4.4x3.6mm_P2.54mm, F.Cu at (140.5, 81.5)
- added U6: LTV-357T, Package_SO:SO-4_4.4x3.6mm_P2.54mm, F.Cu at (219.8, 102.0)
- added U6: LTV-357T, Package_SO:SO-4_4.4x3.6mm_P2.54mm, F.Cu at (140.8, 76.5)
- added U7: LTV-357T, Package_SO:SO-4_4.4x3.6mm_P2.54mm, F.Cu at (224.7, 114.2)
- added U8: LTV-357T, Package_SO:SO-4_4.4x3.6mm_P2.54mm, F.Cu at (224.7, 119.5)
- added U9: LTV-357T, Package_SO:SO-4_4.4x3.6mm_P2.54mm, F.Cu at (129.0, 78.2)
- J1, J11, J2, J3, J4: footprint TerminalBlock_Phoenix:TerminalBlock_Phoenix_MKDS-1,5-2-5.08_1x02_P5.08mm_Horizontal -> TerminalBlock_Phoenix:TerminalBlock_Phoenix_MPT-0,5-2-2.54_1x02_P2.54mm_Horizontal
- J10: value Screw_Terminal_01x02 -> Relay; footprint TerminalBlock_Phoenix:TerminalBlock_Phoenix_MKDS-1,5-2-5.08_1x02_P5.08mm_Horizontal -> TerminalBlock_Phoenix:TerminalBlock_Phoenix_MPT-0,5-6-2.54_1x06_P2.54mm_Horizontal
- J5: value Relay -> Entrada An 5-20mA; footprint TerminalBlock_Phoenix:TerminalBlock_Phoenix_MKDS-1,5-6_1x06_P5.00mm_Horizontal -> TerminalBlock_Phoenix:TerminalBlock_Phoenix_MPT-0,5-2-2.54_1x02_P2.54mm_Horizontal
- J6: value Entrada An 4-20mA -> PNP OUTPUT; footprint TerminalBlock_Phoenix:TerminalBlock_Phoenix_MKDS-1,5-2-5.08_1x02_P5.08mm_Horizontal -> TerminalBlock_Phoenix:TerminalBlock_Phoenix_MPT-0,5-2-2.54_1x02_P2.54mm_Horizontal
- J7: value Salida An 4-20mA -> NPN OUTPUT; footprint TerminalBlock_Phoenix:TerminalBlock_Phoenix_MKDS-1,5-2-5.08_1x02_P5.08mm_Horizontal -> TerminalBlock_Phoenix:TerminalBlock_Phoenix_MPT-0,5-2-2.54_1x02_P2.54mm_Horizontal
- J8: value Salida An 0-10V -> Salidas An; footprint TerminalBlock_Phoenix:TerminalBlock_Phoenix_MKDS-1,5-3-5.08_1x03_P5.08mm_Horizontal -> TerminalBlock_Phoenix:TerminalBlock_Phoenix_MPT-0,5-2-2.54_1x02_P2.54mm_Horizontal
- J9: footprint TerminalBlock_Phoenix:TerminalBlock_Phoenix_MKDS-1,5-3-5.08_1x03_P5.08mm_Horizontal -> TerminalBlock_Phoenix:TerminalBlock_Phoenix_MPT-0,5-3-2.54_1x03_P2.54mm_Horizontal
- moved J10 130.4 mm to (104.3, 144.5), turned to 0 degrees
- moved J5 110.8 mm to (114.0, 69.5), turned to 180 degrees
- moved C1 103.9 mm to (232.9, 124.3)
- moved R1 103.9 mm to (232.9, 126.1)
- moved J11 102.7 mm to (97.5, 144.5)
- moved J9 66.4 mm to (121.4, 144.5)
- moved J4 53.5 mm to (120.9, 69.5)
- moved J8 46.5 mm to (131.0, 144.5)
- moved J3 42.3 mm to (128.0, 69.5)
- moved J1 41.8 mm to (141.9, 69.5)
- moved J2 38.0 mm to (134.9, 69.5)
- moved J7 37.4 mm to (137.7, 144.5)
- moved J6 36.1 mm to (144.5, 144.5)
- moved U1 17.7 mm to (173.2, 109.8), turned to -90 degrees
Connections:
- C1 pad 1: Net-(U1-EN) -> GND
- C1 pad 2: GND -> Net-(U1-EN)
- J10 pad 1: /board_zorion/D_IN_1 -> /board_zorion/RLY1_C
- J10 pad 2: /board_zorion/D_IN_2 -> /board_zorion/RLY1_NC
- J5 pad 1: /board_zorion/RLY1_C -> /board_zorion/A_IN_420mA
- J5 pad 2: /board_zorion/RLY1_NC -> GND
- J6 pad 1: /board_zorion/A_IN_420mA -> /board_zorion/PNP_OUT_1
- J6 pad 2: GND -> /board_zorion/PNP_OUT_2
- J7 pad 1: /board_zorion/A_OUT_420mA -> /board_zorion/NPN_OUT_1
- J7 pad 2: GND -> /board_zorion/NPN_OUT_2
- J8 pad 1: unconnected-(J8-Pin_1-Pad1) -> /board_zorion/A_An_OUT
- J8 pad 2: /board_zorion/A_OUT_10V -> /board_zorion/V_An_OUT
- J9 pad 1: /board_zorion/RS485_A -> /board_zorion/RS485_B
- J9 pad 2: /board_zorion/RS485_B -> GND
- J9 pad 3: GND -> /board_zorion/RS485_A
- U1 pad 12: unconnected-(U1-IO8-Pad12) -> /board_zorion/A_IN_32V/32V_A_IN_IN
- U1 pad 13: unconnected-(U1-USB_D--Pad13) -> /board_zorion/A_IN_10V/10V_A_IN_OUT
- U1 pad 14: unconnected-(U1-USB_D+-Pad14) -> /board_zorion/A_IN_420mA
- U1 pad 15: unconnected-(U1-IO3-Pad15) -> /board_zorion/Rele_IN/RELAY1_IN
- U1 pad 16: unconnected-(U1-IO46-Pad16) -> /board_zorion/Rele_IN/RELAY2_IN
- U1 pad 17: unconnected-(U1-IO9-Pad17) -> /board_zorion/RS485_driver/RS485_IN
- U1 pad 18: unconnected-(U1-IO10-Pad18) -> /board_zorion/RS485_driver/RS485_OUT
- U1 pad 34: unconnected-(U1-IO41-Pad34) -> /board_zorion/Ma_OUT/SLCLK
- U1 pad 35: unconnected-(U1-IO42-Pad35) -> /board_zorion/Ma_OUT/SDA
- U1 pad 36: /board_zorion/RS485_driver/RS485_OUT -> unconnected-(U1-U0RXD/GPIO44/CLK_OUT2-Pad36)
- U1 pad 37: /board_zorion/RS485_driver/RS485_IN -> unconnected-(U1-U0TXD/GPIO43/CLK_OUT1-Pad37)
- U1 pad 6: unconnected-(U1-IO6-Pad6) -> /board_zorion/NPN_IN/NPN_IN_IN_1
- U1 pad 7: unconnected-(U1-IO7-Pad7) -> /board_zorion/NPN_IN/NPN_IN_IN_2
- U1 pad 8: unconnected-(U1-IO15-Pad8) -> /board_zorion/PNP_IN/PNP_IN_IN_1
- U1 pad 9: unconnected-(U1-IO16-Pad9) -> /board_zorion/PNP_IN/PNP_IN_IN_2
Routing:
- net GND: track 0.00 -> 164.7 mm
- net /board_zorion/RLY2_NO: track 0.00 -> 77.9 mm
- net /board_zorion/A_IN_420mA: track 0.00 -> 75.7 mm
- net /board_zorion/A_IN_10V/10V_A_IN_OUT: track 0.00 -> 67.1 mm
- net /board_zorion/Rele_IN/RELAY2_IN: track 0.00 -> 64.9 mm
- net VCC: track 0.00 -> 64.2 mm
- net /board_zorion/Rele_IN/RELAY1_IN: track 0.00 -> 63.0 mm
- net /board_zorion/A_IN_32V/32V_A_IN_IN: track 0.00 -> 55.9 mm
- net /board_zorion/RLY2_NC: track 0.00 -> 55.0 mm
- net /board_zorion/PNP_IN/PNP_IN_IN_2: track 0.00 -> 53.8 mm
- net /board_zorion/PNP_IN/PNP_IN_IN_1: track 0.00 -> 52.8 mm
- net /board_zorion/RLY1_NC: track 0.00 -> 48.4 mm
- net /board_zorion/RLY1_NO: track 0.00 -> 46.9 mm
- net /board_zorion/RS485_driver/RS485_IN: track 0.00 -> 43.7 mm
- net /board_zorion/RS485_driver/RS485_OUT: track 0.00 -> 40.6 mm
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
Commit message: Actualizacion 5
Parts:
- added C10: 100nF, Capacitor_SMD:C_0201_0603Metric, F.Cu at (155.0, 133.8)
- added C11: 1uF, Capacitor_SMD:C_0201_0603Metric, F.Cu at (155.0, 135.5)
- added C12: 220pF, Capacitor_SMD:C_0201_0603Metric, F.Cu at (140.3, 134.6)
- added R24: 4.7K, Resistor_SMD:R_0201_0603Metric, F.Cu at (140.3, 136.0)
- added R25: 10K, Resistor_SMD:R_0201_0603Metric, F.Cu at (140.3, 137.5)
- added R26: 4.7K, Resistor_SMD:R_0201_0603Metric, F.Cu at (140.3, 133.0)
- added R27: 10K, Resistor_SMD:R_0201_0603Metric, F.Cu at (133.3, 135.0)
- added R28: 10K, Resistor_SMD:R_0201_0603Metric, F.Cu at (133.3, 136.0)
- added R29: 2.5K, Resistor_SMD:R_0201_0603Metric, F.Cu at (133.3, 137.5)
- added U11: ~, Proyecto_componente:GP8201S, F.Cu at (149.5, 135.5)
- added U12: ~, Proyecto_componente:GP8303, F.Cu at (137.0, 136.0)
- moved Q2 72.5 mm to (143.8, 117.7)
- moved Q1 20.5 mm to (153.0, 117.5)
- moved C1 8.59 mm to (238.0, 131.2)
- moved R1 8.59 mm to (238.0, 133.0)
- moved U5 4.07 mm to (216.7, 99.2)
- moved U6 4.07 mm to (216.7, 104.5)
Connections:
- U1 pad 19: unconnected-(U1-GPIO11/TOUCH11/ADC2_CH0/FSPID/FSPIIO5/SUBSPID-Pad19) -> /board_zorion/NPN_OUT/NPN_OUT_IN_1
- U1 pad 20: unconnected-(U1-GPIO12/TOUCH12/ADC2_CH1/FSPICLK/FSPIIO6/SUBSPICLK-Pad20) -> /board_zorion/NPN_OUT/NPN_OUT_IN_2
Routing:
- net /board_zorion/Ma_OUT/SDA: track 0.00 -> 45.4 mm
- net /board_zorion/Ma_OUT/SLCLK: track 0.00 -> 37.3 mm
- net /board_zorion/A_An_OUT: track 0.00 -> 22.4 mm, vias 0 -> 1
- net Net-(U12-V5V): track 0.00 -> 21.8 mm
- net GND: track 164.7 -> 184.4 mm
- net Net-(U12-SET): track 0.00 -> 16.7 mm
- net Net-(U12-A2): track 0.00 -> 8.66 mm
- net Net-(U12-A1): track 0.00 -> 7.45 mm
- net Net-(U12-A0): track 0.00 -> 5.39 mm
- net +3.3V: track 1.50 -> 5.97 mm
