File: micro_puerta/micro_puerta.kicad_pcb (KiCad board)
At the start: 2 copper layers, 62 parts, among them J1 Entrada NPN, J10 Relay, J11 Screw_Terminal_01x02, J2 Entradas PNP, J3 Entrada An 0-32V, J4 Entrada An 0-10V, J5 Entrada An 5-20mA, J6 PNP OUTPUT, J7 NPN OUTPUT, J8 Salidas An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

Commit message: Actualizacion 7
Parts:
- removed U2: AP63200WU, Package_TO_SOT_SMD:TSOT-23-6
- added R12: 100, Resistor_SMD:R_0201_0603Metric, F.Cu at (173.8, 128.5)
- added R13: 1k, Resistor_SMD:R_0201_0603Metric, F.Cu at (166.8, 128.3)
- added R14: 100, Resistor_SMD:R_0201_0603Metric, F.Cu at (173.8, 131.0)
- added R15: 1k, Resistor_SMD:R_0201_0603Metric, F.Cu at (166.8, 130.5)
- added R2: 2.2K, Resistor_SMD:R_0201_0603Metric, F.Cu at (146.0, 131.0)
- moved R1 75.7 mm to (172.5, 95.0)
- moved C1 72.3 mm to (176.0, 94.0)
- moved U8 59.0 mm to (170.0, 141.5), turned to 90 degrees
- moved U7 57.7 mm to (170.0, 132.5), turned to 90 degrees
- moved Q4 55.9 mm to (162.0, 142.0), turned to -90 degrees
- moved Q3 50.7 mm to (162.0, 132.5), turned to -90 degrees
- moved Q1 16.7 mm to (154.0, 131.5)
- moved Q2 5.02 mm to (154.0, 141.0)
- moved U1 2.10 mm to (171.2, 109.6)
Connections:
- Q3 pad 3: GNDPWR -> GND
- Q4 pad 3: GNDPWR -> GND
- U1 pad 19: /board_zorion/NPN_OUT/NPN_OUT_IN_1 -> unconnected-(U1-GPIO11/TOUCH11/ADC2_CH0/FSPID/FSPIIO5/SUBSPID-Pad19)
- U1 pad 20: /board_zorion/NPN_OUT/NPN_OUT_IN_2 -> unconnected-(U1-GPIO12/TOUCH12/ADC2_CH1/FSPICLK/FSPIIO6/SUBSPICLK-Pad20)
- U1 pad 36: unconnected-(U1-U0RXD/GPIO44/CLK_OUT2-Pad36) -> /board_zorion/NPN_OUT/NPN_OUT_IN_1
- U1 pad 37: unconnected-(U1-U0TXD/GPIO43/CLK_OUT1-Pad37) -> /board_zorion/NPN_OUT/NPN_OUT_IN_2
- U1 pad 38: unconnected-(U1-GPIO2/TOUCH2/ADC1_CH1-Pad38) -> /board_zorion/PNP_OUT/PNP_OUT_IN_1
- U1 pad 39: unconnected-(U1-GPIO1/TOUCH1/ADC1_CH0-Pad39) -> /board_zorion/PNP_OUT/PNP_OUT_IN_2
- U10 pad 2: GNDPWR -> GND
- U12 pad 5: VCC -> unconnected-(U12-VCC-Pad5)
- U5 pad 2: GNDPWR -> GND
- U6 pad 2: GNDPWR -> GND
- U7 pad 1: Net-(R12-Pad2) -> +3.3V
- U7 pad 2: unconnected-(U7-Pad2) -> Net-(R12-Pad2)
- U7 pad 4: +3.3V -> VCC
- U8 pad 1: Net-(R14-Pad2) -> +3.3V
- U8 pad 2: unconnected-(U8-Pad2) -> Net-(R14-Pad2)
- U8 pad 4: +3.3V -> VCC
- U9 pad 2: GNDPWR -> GND
Routing:
- net +3.3V: track 5.97 -> 208.9 mm, vias 0 -> 6
- net GND: track 192.4 -> 271.8 mm, vias 0 -> 8
- net VCC: track 64.2 -> 118.8 mm, vias 0 -> 2
- net Net-(Q4-G): track 0.00 -> 30.9 mm
- net /board_zorion/NPN_OUT/NPN_OUT_IN_2: track 0.00 -> 30.2 mm
- net /board_zorion/A_IN_32V: track 3.47 -> 30.2 mm
- net /board_zorion/NPN_OUT_1: track 0.00 -> 26.4 mm
- net /board_zorion/PNP_OUT_1: track 0.00 -> 21.2 mm
- net /board_zorion/NPN_OUT/NPN_OUT_IN_1: track 0.00 -> 21.1 mm
- net /board_zorion/NPN_OUT_2: track 0.00 -> 17.7 mm
- net /board_zorion/PNP_OUT_2: track 0.00 -> 15.6 mm
- net Net-(R14-Pad2): track 0.00 -> 14.8 mm
- net /board_zorion/PNP_OUT/PNP_OUT_IN_2: track 0.00 -> 13.3 mm
- net Net-(U1-EN): track 0.00 -> 12.1 mm, vias 0 -> 2
- net /board_zorion/PNP_OUT/PNP_OUT_IN_1: track 0.00 -> 10.3 mm
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- added copper zone on B.Cu, net GND
