File: micro_puerta/Ma_OUT.kicad_sch (KiCad schematic)
At the start: 6 parts

Commit message: actualizacion placa
Parts:
- added R27, R28, R29: 10K, symbol Device:R
Connections:
- net at C12.1, U13.10 (V5V): now also R27.1, R28.1, R29.2
- net A0: no longer names the net of U13.3 (A0)
- net A0: now also R27.2
- net A1: no longer names the net of U13.4 (A1)
- net A1: now also R28.2
- net A2: no longer names the net of U13.9 (A2)
- net A2: now also R29.1
Other:
- moved on the sheet: C12

Commit message: Actualizacion 4 de proyecto
Parts:
- renumbered C13 to C12, C12 to C13, R31 to R24, R28 to R25, R30 to R26, R29 to R28, R32 to R29, U13 to U12
Changed lines of the file:
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@@
 		(on_board yes)
 		(dnp no)
-		(property "Reference" "R28"
+		(property "Reference" "R25"
 			(at 109.22 88.138 90)
 			(effects
@@
 			(project "micro_puerta"
 				(path "/ab2f26d1-d065-4d9e-8f9a-0ccfc45c4b5b/f046d5e0-b81e-417d-b1cc-4f018da2dc07/a2de9f29-1d10-44cf-acd6-187b0a46ed3b"
-					(reference "R28")
+					(reference "R25")
 					(unit 1)
 				)
@@
 		(dnp no)
 		(fields_autoplaced yes)
-		(property "Reference" "#PWR051"
+		(property "Reference" "#PWR049"
 			(at 153.67 101.6 0)
 			(effects
@@
 			(project ""
 				(path "/ab2f26d1-d065-4d9e-8f9a-0ccfc45c4b5b/f046d5e0-b81e-417d-b1cc-4f018da2dc07/a2de9f29-1d10-44cf-acd6-187b0a46ed3b"
-					(reference "#PWR051")
+					(reference "#PWR049")
 					(unit 1)
 				)
@@
 		(dnp no)
 		(fields_autoplaced yes)
-		(property "Reference" "#PWR049"
+		(property "Reference" "#PWR048"
 			(at 119.38 63.5 0)
 			(effects
@@
 			(project ""
 				(path "/ab2f26d1-d065-4d9e-8f9a-0ccfc45c4b5b/f046d5e0-b81e-417d-b1cc-4f018da2dc07/a2de9f29-1d10-44cf-acd6-187b0a46ed3b"
-					(reference "#PWR049")
+					(reference "#PWR048")
 					(unit 1)
 				)
@@
 		(dnp no)
 		(fields_autoplaced yes)
-		(property "Reference" "R30"
+		(property "Reference" "R26"
 			(at 121.92 66.0399 0)
 			(effects
@@
 			(project ""
 				(path "/ab2f26d1-d065-4d9e-8f9a-0ccfc45c4b5b/f046d5e0-b81e-417d-b1cc-4f018da2dc07/a2de9f29-1d10-44cf-acd6-187b0a46ed3b"
-					(reference "R30")
+					(reference "R26")
 					(unit 1)
 				)
@@
 		(dnp no)
 		(fields_autoplaced yes)
-		(property "Reference" "#PWR052"
+		(property "Reference" "#PWR050"
 			(at 162.56 104.14 0)
 			(effects
@@
 			(project ""
 				(path "/ab2f26d1-d065-4d9e-8f9a-0ccfc45c4b5b/f046d5e0-b81e-417d-b1cc-4f018da2dc07/a2de9f29-1d10-44cf-acd6-187b0a46ed3b"
-					(reference "#PWR052")
+					(reference "#PWR050")
 					(unit 1)
 				)
@@
 		(dnp no)
 		(fields_autoplaced yes)
-		(property "Reference" "#PWR053"
+		(property "Reference" "#PWR052"
 			(at 176.53 104.14 0)
 			(effects
@@
 			(project ""
 				(path "/ab2f26d1-d065-4d9e-8f9a-0ccfc45c4b5b/f046d5e0-b81e-417d-b1cc-4f018da2dc07/a2de9f29-1d10-44cf-acd6-187b0a46ed3b"
-					(reference "#PWR053")
+					(reference "#PWR052")
 					(unit 1)
 				)
@@
 		(dnp no)
 		(fields_autoplaced yes)
-		(property "Reference" "R32"
+		(property "Reference" "R29"
 			(at 179.07 92.7099 0)
 			(effects
@@
 			(project ""
 				(path "/ab2f26d1-d065-4d9e-8f9a-0ccfc45c4b5b/f046d5e0-b81e-417d-b1cc-4f018da2dc07/a2de9f29-1d10-44cf-acd6-187b0a46ed3b"
-					(reference "R32")
+					(reference "R29")
 					(unit 1)
 				)
@@
 		(dnp no)
 		(fields_autoplaced yes)
-		(property "Reference" "#PWR048"
+		(property "Reference" "#PWR047"
 			(at 106.68 63.5 0)
 			(effects
@@
 			(project ""
 				(path "/ab2f26d1-d065-4d9e-8f9a-0ccfc45c4b5b/f046d5e0-b81e-417d-b1cc-4f018da2dc07/a2de9f29-1d10-44cf-acd6-187b0a46ed3b"
-					(reference "#PWR048")
+					(reference "#PWR047")
 					(unit 1)
 				)
@@
 		(dnp no)
 		(fields_autoplaced yes)
-		(property "Reference" "C13"
+		(property "Reference" "C12"
 			(at 166.37 92.7099 0)
 			(effects
@@
 			(project ""
 				(path "/ab2f26d1-d065-4d9e-8f9a-0ccfc45c4b5b/f046d5e0-b81e-417d-b1cc-4f018da2dc07/a2de9f29-1d10-44cf-acd6-187b0a46ed3b"
-					(reference "C13")
+					(reference "C12")
 					(unit 1)
 				)
@@
 		(dnp no)
 		(fields_autoplaced yes)
-		(property "Reference" "C12"
+		(property "Reference" "C13"
 			(at 168.91 71.12 90)
 			(effects
@@
 			(project ""
 				(path "/ab2f26d1-d065-4d9e-8f9a-0ccfc45c4b5b/f046d5e0-b81e-417d-b1cc-4f018da2dc07/a2de9f29-1d10-44cf-acd6-187b0a46ed3b"
-					(reference "C12")
+					(reference "C13")
 					(unit 1)
 				)
@@
 		(on_board yes)
 		(dnp no)
-		(property "Reference" "R29"
+		(property "Reference" "R28"
 			(at 154.94 80.264 90)
 			(effects
@@
 			(project "micro_puerta"
 				(path "/ab2f26d1-d065-4d9e-8f9a-0ccfc45c4b5b/f046d5e0-b81e-417d-b1cc-4f018da2dc07/a2de9f29-1d10-44cf-acd6-187b0a46ed3b"
-					(reference "R29")
+					(reference "R28")
 					(unit 1)
 				)
@@
 		(dnp no)
 		(fields_autoplaced yes)
-		(property "Reference" "#PWR050"
+		(property "Reference" "#PWR051"
 			(at 175.26 86.36 0)
 			(effects
@@
 			(project ""
 				(path "/ab2f26d1-d065-4d9e-8f9a-0ccfc45c4b5b/f046d5e0-b81e-417d-b1cc-4f018da2dc07/a2de9f29-1d10-44cf-acd6-187b0a46ed3b"
-					(reference "#PWR050")
+					(reference "#PWR051")
 					(unit 1)
 				)
@@
 		(dnp no)
 		(fields_autoplaced yes)
-		(property "Reference" "R31"
+		(property "Reference" "R24"
 			(at 109.22 66.0399 0)
 			(effects
@@
 			(project ""
 				(path "/ab2f26d1-d065-4d9e-8f9a-0ccfc45c4b5b/f046d5e0-b81e-417d-b1cc-4f018da2dc07/a2de9f29-1d10-44cf-acd6-187b0a46ed3b"
-					(reference "R31")
+					(reference "R24")
 					(unit 1)
 				)
@@
 		(dnp no)
 		(fields_autoplaced yes)
-		(property "Reference" "U13"
+		(property "Reference" "U12"
 			(at 139.7 71.12 0)
 			(effects
@@
 			(project ""
 				(path "/ab2f26d1-d065-4d9e-8f9a-0ccfc45c4b5b/f046d5e0-b81e-417d-b1cc-4f018da2dc07/a2de9f29-1d10-44cf-acd6-187b0a46ed3b"
-					(reference "U13")
-					(unit 1)
-				)
+					(reference "U12")
+					(unit 1)
+				)

Commit message: Actualizacion 5
Parts:
- C12: footprint (none) -> Capacitor_SMD:C_0201_0603Metric
- R24, R25, R26, R27, R28, R29: footprint (none) -> Resistor_SMD:R_0201_0603Metric
- U12: footprint (none) -> Proyecto_componente:GP8303
Connections:
- net VCC: now reaches U12.5 (VCC)
Changed lines of the file:
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@@
+		)
+	)
+	(wire
+		(pts
+			(xy 121.92 93.98) (xy 129.54 93.98)
+		)
+		(stroke
+			(width 0)
+			(type default)
 		)
 	)
@@
 			)
 		)
-		(property "Footprint" ""
+		(property "Footprint" "Resistor_SMD:R_0201_0603Metric"
 			(at 109.22 91.948 90)
 			(effects
@@
 			)
 		)
-		(property "Footprint" ""
+		(property "Footprint" "Resistor_SMD:R_0201_0603Metric"
 			(at 121.158 67.31 90)
 			(effects
@@
 			)
 		)
-		(property "Footprint" ""
+		(property "Footprint" "Resistor_SMD:R_0201_0603Metric"
 			(at 174.752 93.98 90)
 			(effects
@@
 			)
 		)
-		(property "Footprint" ""
+		(property "Footprint" "Capacitor_SMD:C_0201_0603Metric"
 			(at 163.5252 97.79 0)
 			(effects
@@
 			)
 		)
-		(property "Footprint" ""
+		(property "Footprint" "Resistor_SMD:R_0201_0603Metric"
 			(at 121.92 88.138 90)
 			(effects
@@
 			)
 		)
-		(property "Footprint" ""
+		(property "Footprint" "Resistor_SMD:R_0201_0603Metric"
 			(at 154.94 84.328 90)
 			(effects
@@
 	)
 	(symbol
+		(lib_id "power:VCC")
+		(at 121.92 93.98 90)
+		(unit 1)
+		(exclude_from_sim no)
+		(in_bom yes)
+		(on_board yes)
+		(dnp no)
+		(fields_autoplaced yes)
+		(property "Reference" "#PWR012"
+			(at 125.73 93.98 0)
+			(effects
+				(font
+					(size 1.27 1.27)
+				)
+				(hide yes)
+			)
+		)
+		(property "Value" "VCC"
+			(at 118.11 93.9799 90)
+			(effects
+				(font
+					(size 1.27 1.27)
+				)
+				(justify left)
+			)
+		)
+		(property "Footprint" ""
+			(at 121.92 93.98 0)
+			(effects
+				(font
+					(size 1.27 1.27)
+				)
+				(hide yes)
+			)
+		)
+		(property "Datasheet" ""
+			(at 121.92 93.98 0)
+			(effects
+				(font
+					(size 1.27 1.27)
+				)
+				(hide yes)
+			)
+		)
+		(property "Description" "Power symbol creates a global label with name \"VCC\""
+			(at 121.92 93.98 0)
+			(effects
+				(font
+					(size 1.27 1.27)
+				)
+				(hide yes)
+			)
+		)
+		(pin "1"
+		)
+		(instances
+			(project ""
+				(path "/ab2f26d1-d065-4d9e-8f9a-0ccfc45c4b5b/f046d5e0-b81e-417d-b1cc-4f018da2dc07/a2de9f29-1d10-44cf-acd6-187b0a46ed3b"
+					(reference "#PWR012")
+					(unit 1)
+				)
+			)
+		)
+	)
+	(symbol
 		(lib_id "Device:R")
 		(at 106.68 67.31 0)
@@
 			)
 		)
-		(property "Footprint" ""
+		(property "Footprint" "Resistor_SMD:R_0201_0603Metric"
 			(at 104.902 67.31 90)
 			(effects
@@
 			)
 		)
-		(property "Footprint" ""
+		(property "Footprint" "Proyecto_componente:GP8303"
 			(at 139.7 86.36 0)
 			(effects

Commit message: Actualizacion 6
Connections:
- net VCC: no longer names the net of U12.5 (VCC)
Changed lines of the file:
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@@
-		)
-	)
-	(wire
-		(pts
-			(xy 121.92 93.98) (xy 129.54 93.98)
-		)
-		(stroke
-			(width 0)
-			(type default)
 		)
 	)
@@
 					(unit 1)
 				)
-			)
-		)
-	)
-	(symbol
-		(lib_id "power:VCC")
-		(at 121.92 93.98 90)
-		(unit 1)
-		(exclude_from_sim no)
-		(in_bom yes)
-		(on_board yes)
-		(dnp no)
-		(fields_autoplaced yes)
-		(property "Reference" "#PWR012"
-			(at 125.73 93.98 0)
-			(effects
-				(font
-					(size 1.27 1.27)
-				)
-				(hide yes)
-			)
-		)
-		(property "Value" "VCC"
-			(at 118.11 93.9799 90)
-			(effects
-				(font
-					(size 1.27 1.27)
-				)
-				(justify left)
-			)
-		)
-		(property "Footprint" ""
-			(at 121.92 93.98 0)
-			(effects
-				(font
-					(size 1.27 1.27)
-				)
-				(hide yes)
-			)
-		)
-		(property "Datasheet" ""
-			(at 121.92 93.98 0)
-			(effects
-				(font
-					(size 1.27 1.27)
-				)
-				(hide yes)
-			)
-		)
-		(property "Description" "Power symbol creates a global label with name \"VCC\""
-			(at 121.92 93.98 0)
-			(effects
-				(font
-					(size 1.27 1.27)
-				)
-				(hide yes)
-			)
-		)
-		(pin "1"
-		)
-		(instances
-			(project ""
-				(path "/ab2f26d1-d065-4d9e-8f9a-0ccfc45c4b5b/f046d5e0-b81e-417d-b1cc-4f018da2dc07/a2de9f29-1d10-44cf-acd6-187b0a46ed3b"
-					(reference "#PWR012")
-					(unit 1)
-				)
