File: micro_puerta/PNP_OUT.kicad_sch (KiCad schematic)
At the start: 8 parts, among them Q3 NCV8402xST, Q4 NCV8402xST, U8 LTV-357T, U9 LTV-357T

Commit message: Actualizacion 4 de proyecto
Parts:
- renumbered R15 to R12, R16 to R13, R17 to R14, R18 to R15, U8 to U7, U9 to U8
Changed lines of the file:
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@@
 		(dnp no)
 		(fields_autoplaced yes)
-		(property "Reference" "#PWR032"
+		(property "Reference" "#PWR034"
 			(at 214.63 102.87 0)
 			(effects
@@
 			(project "micro_puerta"
 				(path "/ab2f26d1-d065-4d9e-8f9a-0ccfc45c4b5b/f046d5e0-b81e-417d-b1cc-4f018da2dc07/f7dc82f5-2729-4d1a-b9b8-25038fee8530"
-					(reference "#PWR032")
+					(reference "#PWR034")
 					(unit 1)
 				)
@@
 		(dnp no)
 		(fields_autoplaced yes)
-		(property "Reference" "U8"
+		(property "Reference" "U7"
 			(at 87.63 62.23 0)
 			(effects
@@
 			(project "micro_puerta"
 				(path "/ab2f26d1-d065-4d9e-8f9a-0ccfc45c4b5b/f046d5e0-b81e-417d-b1cc-4f018da2dc07/f7dc82f5-2729-4d1a-b9b8-25038fee8530"
-					(reference "U8")
+					(reference "U7")
 					(unit 1)
 				)
@@
 		(dnp no)
 		(fields_autoplaced yes)
-		(property "Reference" "#NPN_VCC03"
+		(property "Reference" "#NPN_VCC02"
 			(at 201.93 67.31 0)
 			(effects
@@
 			(project "micro_puerta"
 				(path "/ab2f26d1-d065-4d9e-8f9a-0ccfc45c4b5b/f046d5e0-b81e-417d-b1cc-4f018da2dc07/f7dc82f5-2729-4d1a-b9b8-25038fee8530"
-					(reference "#NPN_VCC03")
+					(reference "#NPN_VCC02")
 					(unit 1)
 				)
@@
 		(dnp no)
 		(fields_autoplaced yes)
-		(property "Reference" "R16"
+		(property "Reference" "R13"
 			(at 101.6 88.8999 0)
 			(effects
@@
 			(project "micro_puerta"
 				(path "/ab2f26d1-d065-4d9e-8f9a-0ccfc45c4b5b/f046d5e0-b81e-417d-b1cc-4f018da2dc07/f7dc82f5-2729-4d1a-b9b8-25038fee8530"
-					(reference "R16")
+					(reference "R13")
 					(unit 1)
 				)
@@
 		(dnp no)
 		(fields_autoplaced yes)
-		(property "Reference" "R15"
+		(property "Reference" "R12"
 			(at 72.39 62.23 90)
 			(effects
@@
 			(project "micro_puerta"
 				(path "/ab2f26d1-d065-4d9e-8f9a-0ccfc45c4b5b/f046d5e0-b81e-417d-b1cc-4f018da2dc07/f7dc82f5-2729-4d1a-b9b8-25038fee8530"
-					(reference "R15")
+					(reference "R12")
 					(unit 1)
 				)
@@
 		(dnp no)
 		(fields_autoplaced yes)
-		(property "Reference" "#PWR031"
+		(property "Reference" "#PWR033"
 			(at 109.22 102.87 0)
 			(effects
@@
 			(project "micro_puerta"
 				(path "/ab2f26d1-d065-4d9e-8f9a-0ccfc45c4b5b/f046d5e0-b81e-417d-b1cc-4f018da2dc07/f7dc82f5-2729-4d1a-b9b8-25038fee8530"
-					(reference "#PWR031")
+					(reference "#PWR033")
 					(unit 1)
 				)
@@
 		(dnp no)
 		(fields_autoplaced yes)
-		(property "Reference" "R17"
+		(property "Reference" "R14"
 			(at 177.8 62.23 90)
 			(effects
@@
 			(project "micro_puerta"
 				(path "/ab2f26d1-d065-4d9e-8f9a-0ccfc45c4b5b/f046d5e0-b81e-417d-b1cc-4f018da2dc07/f7dc82f5-2729-4d1a-b9b8-25038fee8530"
-					(reference "R17")
+					(reference "R14")
 					(unit 1)
 				)
@@
 		(dnp no)
 		(fields_autoplaced yes)
-		(property "Reference" "U9"
+		(property "Reference" "U8"
 			(at 193.04 62.23 0)
 			(effects
@@
 			(project "micro_puerta"
 				(path "/ab2f26d1-d065-4d9e-8f9a-0ccfc45c4b5b/f046d5e0-b81e-417d-b1cc-4f018da2dc07/f7dc82f5-2729-4d1a-b9b8-25038fee8530"
-					(reference "U9")
+					(reference "U8")
 					(unit 1)
 				)
@@
 		(dnp no)
 		(fields_autoplaced yes)
-		(property "Reference" "#NPN_VCC02"
+		(property "Reference" "#NPN_VCC01"
 			(at 96.52 67.31 0)
 			(effects
@@
 			(project "micro_puerta"
 				(path "/ab2f26d1-d065-4d9e-8f9a-0ccfc45c4b5b/f046d5e0-b81e-417d-b1cc-4f018da2dc07/f7dc82f5-2729-4d1a-b9b8-25038fee8530"
-					(reference "#NPN_VCC02")
+					(reference "#NPN_VCC01")
 					(unit 1)
 				)
@@
 		(dnp no)
 		(fields_autoplaced yes)
-		(property "Reference" "R18"
+		(property "Reference" "R15"
 			(at 207.01 88.8999 0)
 			(effects
@@
 			(project "micro_puerta"
 				(path "/ab2f26d1-d065-4d9e-8f9a-0ccfc45c4b5b/f046d5e0-b81e-417d-b1cc-4f018da2dc07/f7dc82f5-2729-4d1a-b9b8-25038fee8530"
-					(reference "R18")
-					(unit 1)
-				)
+					(reference "R15")
+					(unit 1)
+				)

Commit message: Actualizacion 6
Parts:
- R12, R14: footprint (none) -> Resistor_SMD:R_0201_0603Metric
- R13, R15: value R -> 1k; footprint (none) -> Resistor_SMD:R_0201_0603Metric
Connections:
- net +3.3V: now also U7.1, U8.1; no longer U7.4, U8.4
- net at R12.2: now also U7.2; no longer U7.1
- net at R14.2: now also U8.2; no longer U8.1
- net GNDPWR renamed GND
- new net VCC: U7.4, U8.4
Other:
- moved on the sheet: R12, R14
