File: micro_puerta/V_AN_Out.kicad_sch (KiCad schematic)
At the start: 4 parts

Commit message: Actualizacion 4 de proyecto
Parts:
- renumbered D3 to D2, U12 to U11
Changed lines of the file:
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@@
 		(dnp no)
 		(fields_autoplaced yes)
-		(property "Reference" "U12"
+		(property "Reference" "U11"
 			(at 144.78 77.47 0)
 			(effects
@@
 			(project ""
 				(path "/ab2f26d1-d065-4d9e-8f9a-0ccfc45c4b5b/f046d5e0-b81e-417d-b1cc-4f018da2dc07/4bb98c27-d9bc-476b-8b92-dbb7ee163d5a"
-					(reference "U12")
+					(reference "U11")
 					(unit 1)
 				)
@@
 		(dnp no)
 		(fields_autoplaced yes)
-		(property "Reference" "#PWR028"
+		(property "Reference" "#PWR043"
 			(at 132.08 97.79 0)
 			(effects
@@
 			(project "micro_puerta"
 				(path "/ab2f26d1-d065-4d9e-8f9a-0ccfc45c4b5b/f046d5e0-b81e-417d-b1cc-4f018da2dc07/4bb98c27-d9bc-476b-8b92-dbb7ee163d5a"
-					(reference "#PWR028")
+					(reference "#PWR043")
 					(unit 1)
 				)
@@
 		(dnp no)
 		(fields_autoplaced yes)
-		(property "Reference" "D3"
+		(property "Reference" "D2"
 			(at 173.99 96.5199 90)
 			(effects
@@
 			(project "micro_puerta"
 				(path "/ab2f26d1-d065-4d9e-8f9a-0ccfc45c4b5b/f046d5e0-b81e-417d-b1cc-4f018da2dc07/4bb98c27-d9bc-476b-8b92-dbb7ee163d5a"
-					(reference "D3")
+					(reference "D2")
 					(unit 1)
 				)
@@
 		(dnp no)
 		(fields_autoplaced yes)
-		(property "Reference" "#PWR026"
+		(property "Reference" "#PWR045"
 			(at 175.26 86.36 0)
 			(effects
@@
 			(project "micro_puerta"
 				(path "/ab2f26d1-d065-4d9e-8f9a-0ccfc45c4b5b/f046d5e0-b81e-417d-b1cc-4f018da2dc07/4bb98c27-d9bc-476b-8b92-dbb7ee163d5a"
-					(reference "#PWR026")
+					(reference "#PWR045")
 					(unit 1)
 				)
@@
 		(dnp no)
 		(fields_autoplaced yes)
-		(property "Reference" "#PWR023"
+		(property "Reference" "#PWR044"
 			(at 161.29 110.49 0)
 			(effects
@@
 			(project "micro_puerta"
 				(path "/ab2f26d1-d065-4d9e-8f9a-0ccfc45c4b5b/f046d5e0-b81e-417d-b1cc-4f018da2dc07/4bb98c27-d9bc-476b-8b92-dbb7ee163d5a"
-					(reference "#PWR023")
-					(unit 1)
-				)
+					(reference "#PWR044")
+					(unit 1)
+				)

Commit message: Actualizacion 5
Parts:
- C10, C11: footprint (none) -> Capacitor_SMD:C_0201_0603Metric
- U11: footprint (none) -> Proyecto_componente:GP8201S
Changed lines of the file:
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@@
 			)
 		)
-		(property "Footprint" ""
+		(property "Footprint" "Proyecto_componente:GP8201S"
 			(at 144.78 91.44 0)
 			(effects
@@
 			)
 		)
-		(property "Footprint" ""
+		(property "Footprint" "Capacitor_SMD:C_0201_0603Metric"
 			(at 166.37 85.3948 0)
 			(effects
@@
 			)
 		)
-		(property "Footprint" ""
+		(property "Footprint" "Capacitor_SMD:C_0201_0603Metric"
 			(at 160.3248 93.98 0)
 			(effects

Commit message: Actualizacion 6
Parts:
- C10, C11: footprint Capacitor_SMD:C_0201_0603Metric -> (none)
- U11: footprint Proyecto_componente:GP8201S -> (none)
Changed lines of the file:
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@@
 			)
 		)
-		(property "Footprint" "Proyecto_componente:GP8201S"
+		(property "Footprint" ""
 			(at 144.78 91.44 0)
 			(effects
@@
 			)
 		)
-		(property "Footprint" "Capacitor_SMD:C_0201_0603Metric"
+		(property "Footprint" ""
 			(at 166.37 85.3948 0)
 			(effects
@@
 			)
 		)
-		(property "Footprint" "Capacitor_SMD:C_0201_0603Metric"
+		(property "Footprint" ""
 			(at 160.3248 93.98 0)
 			(effects
