File: micro_puerta/_autosave-micro_puerta.kicad_pcb (KiCad board)
At the start: 2 copper layers, 62 parts, among them J1 Entrada NPN, J10 Relay, J11 Screw_Terminal_01x02, J2 Entradas PNP, J3 Entrada An 0-32V, J4 Entrada An 0-10V, J5 Entrada An 5-20mA, J6 PNP OUTPUT, J7 NPN OUTPUT, J8 Salidas An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

Commit message: Actualizacion 6
Parts:
- added R12: 100, Resistor_SMD:R_0201_0603Metric, F.Cu at (173.8, 128.5)
- added R13: 1k, Resistor_SMD:R_0201_0603Metric, F.Cu at (166.8, 128.3)
- added R14: 100, Resistor_SMD:R_0201_0603Metric, F.Cu at (173.8, 131.0)
- added R15: 1k, Resistor_SMD:R_0201_0603Metric, F.Cu at (166.8, 130.5)
- moved U8 59.0 mm to (170.0, 141.5), turned to 90 degrees
- moved U7 57.7 mm to (170.0, 132.5), turned to 90 degrees
- moved Q4 55.9 mm to (162.0, 142.0), turned to -90 degrees
- moved Q3 50.7 mm to (162.0, 132.5), turned to -90 degrees
- moved C1 19.6 mm to (254.8, 141.2)
- moved R1 19.6 mm to (254.8, 143.0)
- moved Q1 16.7 mm to (154.0, 131.5)
- moved Q2 5.02 mm to (154.0, 141.0)
- moved U1 2.10 mm to (171.2, 109.6)
Connections:
- Q1 pad 1: /board_zorion/NPN_OUT/NPN_OUT_IN_1 -> /board_zorion/A_IN_420mA
- Q3 pad 3: GNDPWR -> GND
- Q4 pad 3: GNDPWR -> GND
- U1 pad 19: /board_zorion/NPN_OUT/NPN_OUT_IN_1 -> unconnected-(U1-GPIO11/TOUCH11/ADC2_CH0/FSPID/FSPIIO5/SUBSPID-Pad19)
- U1 pad 20: /board_zorion/NPN_OUT/NPN_OUT_IN_2 -> unconnected-(U1-GPIO12/TOUCH12/ADC2_CH1/FSPICLK/FSPIIO6/SUBSPICLK-Pad20)
- U1 pad 36: unconnected-(U1-U0RXD/GPIO44/CLK_OUT2-Pad36) -> /board_zorion/A_IN_420mA
- U1 pad 37: unconnected-(U1-U0TXD/GPIO43/CLK_OUT1-Pad37) -> /board_zorion/NPN_OUT/NPN_OUT_IN_2
- U1 pad 38: unconnected-(U1-GPIO2/TOUCH2/ADC1_CH1-Pad38) -> /board_zorion/PNP_OUT/PNP_OUT_IN_1
- U1 pad 39: unconnected-(U1-GPIO1/TOUCH1/ADC1_CH0-Pad39) -> /board_zorion/PNP_OUT/PNP_OUT_IN_2
- U12 pad 5: VCC -> unconnected-(U12-VCC-Pad5)
- U7 pad 1: Net-(R12-Pad2) -> +3.3V
- U7 pad 2: unconnected-(U7-Pad2) -> Net-(R12-Pad2)
- U7 pad 4: +3.3V -> VCC
- U8 pad 1: Net-(R14-Pad2) -> +3.3V
- U8 pad 2: unconnected-(U8-Pad2) -> Net-(R14-Pad2)
- U8 pad 4: +3.3V -> VCC
Routing:
- net /board_zorion/Rele_IN/RELAY1_IN: track 63.0 -> 7.45 mm
- net /board_zorion/Rele_IN/RELAY2_IN: track 64.9 -> 9.89 mm
- net Net-(Q4-G): track 0.00 -> 30.9 mm
- net /board_zorion/RS485_driver/RS485_IN: track 43.7 -> 13.0 mm
- net /board_zorion/RS485_driver/RS485_OUT: track 40.6 -> 11.2 mm
- net /board_zorion/NPN_OUT_1: track 0.00 -> 26.4 mm
- net /board_zorion/NPN_OUT/NPN_OUT_IN_2: track 0.00 -> 21.9 mm
- net /board_zorion/PNP_OUT_1: track 0.00 -> 21.2 mm
- net /board_zorion/NPN_OUT_2: track 0.00 -> 17.7 mm
- net /board_zorion/PNP_OUT_2: track 0.00 -> 15.6 mm
- net Net-(R14-Pad2): track 0.00 -> 14.8 mm
- net GND: track 192.4 -> 204.0 mm
- net /board_zorion/A_IN_420mA: track 75.7 -> 86.5 mm
- net VCC: track 64.2 -> 73.7 mm
- net +3.3V: track 5.97 -> 15.5 mm
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